Commit message: Get the project launch file working and publishing the tf tree

File: ros2_ws/src/companion_trolley_description/urdf/companion_trolley.urdf (robot description, URDF)
Before this commit: robot companion_trolley, 9 links, 8 joints
Joints:
- joint base_left_wheel_joint: axis 0 1 0 -> (none); type continuous -> fixed
- joint base_right_wheel_joint: axis 0 1 0 -> (none); type continuous -> fixed

Commit message: real measurements for URDF file added

File: ros2_ws/src/companion_trolley_description/urdf/companion_trolley.urdf (robot description, URDF)
Before this commit: robot companion_trolley, 9 links, 8 joints
Links:
- added link IMU; visual box size=.02 .025 .001
- link base_link: geometry visual box size=0.443 0.40 0.86
- link caster_wheel_BL: geometry visual sphere radius=0.045
- link caster_wheel_BR: geometry visual sphere radius=0.045
- link caster_wheel_FL: geometry visual sphere radius=0.045
- link caster_wheel_FR: geometry visual sphere radius=0.045
- link left_wheel: geometry visual cylinder length=0.035 radius=0.09
- link right_wheel: geometry visual cylinder length=0.035 radius=0.09
Joints:
- added joint base_IMU_joint: type fixed, parent base_link, child IMU, origin xyz=0.1765 0.01 0.05 rpy=0 0 0
- joint base_caster_wheel_BL_joint: origin xyz=-0.175 -0.1 -0.025 rpy=0 0 0 -> xyz=-0.1765 0.155 -0.045 rpy=0 0 0
- joint base_caster_wheel_BR_joint: origin xyz=-0.175 0.1 -0.025 rpy=0 0 0 -> xyz=-0.1765 -0.155 -0.045 rpy=0 0 0
- joint base_caster_wheel_FL_joint: origin xyz=0.175 -0.1 -0.025 rpy=0 0 0 -> xyz=0.1765 0.155 -0.045 rpy=0 0 0
- joint base_caster_wheel_FR_joint: origin xyz=0.175 0.1 -0.025 rpy=0 0 0 -> xyz=0.1765 -0.155 -0.045 rpy=0 0 0
- joint base_joint: origin xyz=0 0 0.05 rpy=0 0 0 -> xyz=0 0 0.09 rpy=0 0 0
- joint base_left_wheel_joint: origin xyz=0 0.15 0 rpy=0 0 0 -> xyz=0 0.2175 0 rpy=0 0 0
- joint base_lidar_joint: origin xyz=0.18 0 0.1 rpy=0 0 0 -> xyz=-0.1415 0 0.165 rpy=0 0 0
- joint base_right_wheel_joint: origin xyz=0 -0.15 0 rpy=0 0 0 -> xyz=0 -0.2175 0 rpy=0 0 0

Commit message: arduino serial manager setup to read in and publish imu data

File: ros2_ws/src/companion_trolley_description/urdf/companion_trolley.urdf (robot description, URDF)
Before this commit: robot companion_trolley, 10 links, 9 joints
Links:
- removed link IMU
- removed link lidar
- added link imu_link; visual box size=.02 .025 .001
- added link lidar_link; visual cylinder length=0.035 radius=0.02
Joints:
- joint base_IMU_joint: child IMU -> imu_link
- joint base_lidar_joint: child lidar -> lidar_link

Commit message: UWB added into urdf file

File: ros2_ws/src/companion_trolley_description/urdf/companion_trolley.urdf (robot description, URDF)
Before this commit: robot companion_trolley, 10 links, 9 joints
Links:
- added link uwb_link; visual box size=.015 .08 .035
Joints:
- added joint base_UWB_joint: type fixed, parent base_link, child uwb_link, origin xyz=-0.229 -0.01 0.455 rpy=0 0 0
